Commit message: update ros controller

File: dynamics_ws/src/parallel_urdf/urdf/parabot.urdf (robot description, URDF)
Before this commit: robot parabot, 13 links, 12 joints
Links:
- added link base_move; visual box size=0.001 0.001 0.001
Joints:
- added joint floating_base: type fixed, parent base_move, child base, origin xyz=0 0 0 rpy=0 0 0
- joint Jointleft_1: limit lower=0.04 upper=0.3 effort=10 velocity=0.1 -> lower=0.04 upper=0.3 effort=100 velocity=21
- joint Jointright_1: limit lower=0.04 upper=0.3 effort=10 velocity=0.1 -> lower=0.04 upper=0.3 effort=100 velocity=21
- joint Jointup_1: limit lower=0.04 upper=0.3 effort=10 velocity=0.1 -> lower=0.04 upper=0.3 effort=100 velocity=21
- joint Jointup_4: limit lower=-3 upper=3 effort=10 velocity=0.1 -> lower=-0.9 upper=3 effort=10 velocity=0.1
- joint fixed: child base -> base_move
